Commit message: Got lidar working properly by fixing some urdf issues

File: src/lidar_bot_description/urdf/lidar_bot.urdf.xacro (robot description, xacro)
@@ -9,4 +9,7 @@
     <xacro:property name="caster_mass" value="0.001"/>
     <xacro:property name="caster_radius" value="${(turtle_wheel_radius-base_thickness/2.0)/2.0}"/>
+    <xacro:property name="lidar_mass" value="0.001"/>
+    <xacro:property name="lidar_length" value="0.01"/>
+    <xacro:property name="lidar_radius" value="0.01"/>
     <link name="base_link">
         <visual>
@@ -112,4 +115,30 @@
         </inertial>
     </link>
+    <link name="lidar">
+        <visual>
+            <geometry>
+                <cylinder length="${lidar_length}" radius="${lidar_radius}"/>
+            </geometry>
+        </visual>
+        <collision>
+            <geometry>
+                <cylinder length="${lidar_length}" radius="${lidar_radius}"/>
+            </geometry>
+        </collision>
+        <inertial>
+            <mass value="${lidar_mass}"/>
+            <inertia
+                ixx="${(1.0/12.0) * lidar_mass * (3*lidar_radius*lidar_radius + lidar_length*lidar_length)}"
+                iyy="${(1.0/12.0) * lidar_mass * (3*lidar_radius*lidar_radius + lidar_length*lidar_length)}"
+                izz="${0.5 * lidar_mass * lidar_radius*lidar_radius}"
+                ixy="0" ixz="0" iyz="0"/>
+        </inertial>
+    </link>
+    <link name="base_footprint"/>
+    <joint name="footprint_base" type="fixed">
+        <parent link="base_footprint"/>
+        <child link="base_link"/>
+        <origin xyz="0 0 ${base_thickness}" rpy="0 0 0"/>
+    </joint>
     <joint name="base_left_wheel" type="continuous">
         <parent link="base_link"/>
@@ -133,4 +162,10 @@
         <child link="caster_wheel_back"/>
         <origin xyz ="-${base_radius-(base_radius/4)} 0 -${base_thickness/2.0+caster_radius}" rpy="0 0 0"/>
+    </joint>
+    <joint name="base_lidar" type="fixed">
+        <parent link="base_link"/>
+        <child link="lidar"/>
+        <origin xyz="${base_radius-lidar_radius} 0 ${base_thickness/2.0+lidar_length/2.0}"/>
+        <axis xyz="0 1 0" rpy="0 0 0"/>
     </joint>
     <gazebo reference="caster_wheel_front">
@@ -154,5 +189,5 @@
             <!-- output -->
             <frame_id>odom</frame_id>
-            <child_frame_id>base_link</child_frame_id>
+            <child_frame_id>base_footprint</child_frame_id>
         </plugin>
     </gazebo>
@@ -166,3 +201,33 @@
         </plugin>
     </gazebo>
+    <gazebo reference="lidar">
+        <sensor name="gpu_lidar" type="gpu_lidar">
+            <pose relative_to="lidar">0 0 0 0 0 0</pose>
+            <topic>lidar</topic>
+            <update_rate>10</update_rate>
+            <ray>
+                <scan>
+                    <horizontal>
+                        <samples>640</samples>
+                        <resolution>1</resolution>
+                        <min_angle>-1.396263</min_angle>
+                        <max_angle>1.396263</max_angle>
+                    </horizontal>
+                    <vertical>
+                        <samples>1</samples>
+                        <resolution>0.01</resolution>
+                        <min_angle>0</min_angle>
+                        <max_angle>0</max_angle>
+                    </vertical>
+                </scan>
+                <range>
+                    <min>0.08</min>
+                    <max>10.0</max>
+                    <resolution>0.01</resolution>
+                </range>
+            </ray>
+            <always_on>1</always_on>
+            <visualize>true</visualize>
+        </sensor>
+    </gazebo>
 </robot>
